File: MacroPadPCB.kicad_pcb (KiCad board)
At the start: 2 copper layers, 273.8 x 187.3 mm, 24 parts, among them SW1 SW_Push, U1 ATmega32U4-AU, Y1 16MHz

Commit message: Ground filling done - Bug fixing WIP
Routing:
- net Net-(USB1-Pad6): track 0.00 -> 16.3 mm
- added copper zone on F.Cu, net GND
Other:
- board size 273.8 x 187.3 mm -> 87.3 x 46.8 mm
- rule trace_min: 0.2 -> 0.002
- rule via_min_size: 0.4 -> 0.002
- board text added: "Ismael - MacroPad"
